Commit message: changes for ground plane

File: cartographer_ros/urdf/backpack_3d_mrt.urdf (robot description, URDF)
Before this commit: robot cartographer_backpack_3d, 3 links, 2 joints
Links:
- removed link laser
- added link sensor/velodyne; visual cylinder length=0.07 radius=0.05
Joints:
- joint sensor/velodyne_joint: child laser -> sensor/velodyne
